Commit message: proper inertia set but strangly jiggeling

File: jaco_driver/jaco_description/urdf/gazebo/jaco.urdf.xacro (robot description, xacro)
@@ -1,23 +1,13 @@
 <?xml version="1.0"?>
 <robot name="jaco"
-	xmlns:xi="http://www.w3.org/2001/XInclude"
-	xmlns:gazebo="http://playerstage.sourceforge.net/gazebo/xmlschema/#gz"
-	xmlns:model="http://playerstage.sourceforge.net/gazebo/xmlschema/#model"
-	xmlns:sensor="http://playerstage.sourceforge.net/gazebo/xmlschema/#sensor"
-	xmlns:body="http://playerstage.sourceforge.net/gazebo/xmlschema/#body"
-	xmlns:geom="http://playerstage.sourceforge.net/gazebo/xmlschema/#geom"
-	xmlns:joint="http://playerstage.sourceforge.net/gazebo/xmlschema/#joint"
-	xmlns:interface="http://playerstage.sourceforge.net/gazebo/xmlschema/#interface"
-	xmlns:rendering="http://playerstage.sourceforge.net/gazebo/xmlschema/#rendering"
-	xmlns:renderable="http://playerstage.sourceforge.net/gazebo/xmlschema/#renderable"
-	xmlns:controller="http://playerstage.sourceforge.net/gazebo/xmlschema/#controller"
-	xmlns:physics="http://playerstage.sourceforge.net/gazebo/xmlschema/#physics">
+  xmlns:xacro="http://ros.org/wiki/xacro">
+ <xacro:property name="inertia" value="0.001" />
+  <xacro:property name="finger_inertia" value="0.0001" />
 	<gazebo>
-		<!-- controller for the 6 arm joints -->
-		<controller:gazebo_ros_controller_manager name="gazebo_ros_controller_manager" plugin="libgazebo_ros_controller_manager.so">
-		<alwaysOn>true</alwaysOn>
+    <plugin name="gazebo_ros_controller_manager" filename="libgazebo_ros_controller_manager.so">
+      <alwaysOn>true</alwaysOn>
 		<updateRate>1000.0</updateRate>
 		<robotParam>robot_description</robotParam>
-		</controller:gazebo_ros_controller_manager>
+    </plugin>
 	</gazebo>
 	<include filename="$(find jaco_description)/urdf/gazebo/jaco.gazebo.xacro" />
@@ -26,4 +16,5 @@
 	<color rgba="0.2 0.2 0.9 1.0"/>
 	</material>
+	<!--
 	<link name="world"/>
 	<joint name="base_block_joint" type="fixed">
@@ -32,11 +23,12 @@
 		<child link="jaco_base_link" />
 	</joint>
+ -->
 	<!-- The base joint & link -->
 	<link name="jaco_base_link">
 		<inertial>
-			<mass value="6" />
+			<mass value="1" />
 			<!--origin xyz="0 0 -0.0525" rpy="0 0 0"/-->
           		<origin xyz="0 0 0.0" rpy="0 0 0"/>
-			<inertia ixx="100"  ixy="0"  ixz="0" iyy="100" iyz="0" izz="100" />
+			<inertia ixx="${inertia}"  ixy="0"  ixz="0" iyy="${inertia}" iyz="0" izz="${inertia}" />
 		</inertial>
 		<visual>
@@ -67,10 +59,10 @@
 		<parent link="jaco_base_link"/>
 		<child link="jaco_link_1"/>
-		<limit lower="-3.1415926535897931" upper="3.1415926535897931" effort="1" velocity="2.0"/>
+		<limit lower="-3.1415926535897931" upper="3.1415926535897931" effort="30" velocity="5"/>
 	</joint>
 	<link name="jaco_link_1">
 		<inertial>
-			<mass value="4.5"/>
-			<inertia ixx="100.0" ixy="0.0"  ixz="0.0"  iyy="100.0"  iyz="0.0"  izz="100.0" />
+			<mass value="1" />
+			<inertia ixx="${inertia}"  ixy="0"  ixz="0" iyy="${inertia}" iyz="0" izz="${inertia}" />
 			<origin/>
 		</inertial>
@@ -101,10 +93,10 @@
 		<parent link="jaco_link_1"/>
 		<child link="jaco_link_2"/>
-		<limit lower="-3.6651914291881" upper="0.57595865315813" effort="1" velocity="3.1415926535897931"/>
+		<limit lower="-3.6651914291881" upper="0.57595865315813" effort="30" velocity="5"/>
 	</joint>
 	<link name="jaco_link_2">
 		<inertial>
-			<mass value="3.8"/>
-			<inertia ixx="100.0" ixy="0.0"  ixz="0.0"  iyy="100.0"  iyz="0.0"  izz="100.0" />
+			<mass value="1" />
+			<inertia ixx="${inertia}"  ixy="0"  ixz="0" iyy="${inertia}" iyz="0" izz="${inertia}" />
 			<origin/>
 		</inertial>
@@ -135,10 +127,10 @@
 		<parent link="jaco_link_2"/>
 		<child link="jaco_link_3"/>
-		<limit lower="-1.221730476396" upper="4.2935099599061" effort="1" velocity="3.1415926535897931"/>
+		<limit lower="-1.221730476396" upper="4.2935099599061" effort="30" velocity="5"/>
 	</joint>
 	<link name="jaco_link_3">
 		<inertial>
-			<mass value="2"/>
-			<inertia ixx="100.0" ixy="0.0"  ixz="0.0"  iyy="100.0"  iyz="0.0"  izz="100.0" />
+			<mass value="1" />
+			<inertia ixx="${inertia}"  ixy="0"  ixz="0" iyy="${inertia}" iyz="0" izz="${inertia}" />
 			<origin/>
 		</inertial>
@@ -169,10 +161,10 @@
 		<parent link="jaco_link_3"/>
 		<child link="jaco_link_4"/>
-		<limit lower="-3.1415926535897931" upper="3.1415926535897931" effort="1" velocity="2.0"/>
+		<limit lower="-3.1415926535897931" upper="3.1415926535897931" effort="30" velocity="5"/>
 	</joint>
 	<link name="jaco_link_4">
 		<inertial>
-			<mass value="1.5"/>
-			<inertia ixx="100.0" ixy="0.0"  ixz="0.0"  iyy="100.0"  iyz="0.0"  izz="100.0" />
+			<mass value="1" />
+			<inertia ixx="${inertia}"  ixy="0"  ixz="0" iyy="${inertia}" iyz="0" izz="${inertia}" />
 			<origin/>
 		</inertial>
@@ -203,10 +195,10 @@
 		<parent link="jaco_link_4"/>
 		<child link="jaco_link_5"/>
-		<limit lower="-3.1415926535897931" upper="3.1415926535897931" effort="1" velocity="2.0"/>
+		<limit lower="-3.1415926535897931" upper="3.1415926535897931" effort="30" velocity="5"/>
 	</joint>
 	<link name="jaco_link_5">
 		<inertial>
 			<mass value="1.0"/>
-			<inertia ixx="100.0" ixy="0.0"  ixz="0.0"  iyy="100.0"  iyz="0.0"  izz="100.0" />
+			<inertia ixx="${inertia}"  ixy="0"  ixz="0" iyy="${inertia}" iyz="0" izz="${inertia}" />
 			<origin/>
 		</inertial>
@@ -239,10 +231,10 @@
 		<parent link="jaco_link_5"/>
 		<child link="jaco_link_6"/>
-		<limit lower="-3.5415926535897931" upper="3.5415926535897931" effort="1" velocity="2.0"/>
+		<limit lower="-3.5415926535897931" upper="3.5415926535897931" effort="30" velocity="5"/>
 	</joint>
 	<link name="jaco_link_6">
 		<inertial>
-			<mass value="0.8"/>
-			<inertia ixx="100.0" ixy="0.0"  ixz="0.0"  iyy="100.0"  iyz="0.0"  izz="100.0" />
+			<mass value="0.3"/>
+			<inertia ixx="${inertia}"  ixy="0"  ixz="0" iyy="${inertia}" iyz="0" izz="${inertia}" />
 			<origin/>
 		</inertial>
@@ -276,10 +268,10 @@
         <parent link="jaco_link_6"/>
         <child link="jaco_finger_link_1"/>
-		<limit lower="-3.1415926535897931" upper="3.1415926535897931" effort="1" velocity="2.0"/>
+		<limit lower="-3.1415926535897931" upper="3.1415926535897931" effort="30" velocity="5"/>
       </joint>
       <link name="jaco_finger_link_1">
 		<inertial>
 			<mass value="0.05"/>
-			<inertia ixx="10.0" ixy="0.0"  ixz="0.0"  iyy="10.0"  iyz="0.0"  izz="10.0" />
+			<inertia ixx="${finger_inertia}"  ixy="0"  ixz="0" iyy="${finger_inertia}" iyz="0" izz="${finger_inertia}" />
 			<origin/>
 		</inertial>
@@ -310,10 +302,10 @@
         <parent link="jaco_link_6"/>
         <child link="jaco_finger_link_2"/>
-		<limit lower="-3.1415926535897931" upper="3.1415926535897931" effort="1" velocity="2.0"/>
+		<limit lower="-3.1415926535897931" upper="3.1415926535897931" effort="30" velocity="5"/>
       </joint>
       <link name="jaco_finger_link_2">
 		<inertial>
 			<mass value="0.05"/>
-			<inertia ixx="10.0" ixy="0.0"  ixz="0.0"  iyy="10.0"  iyz="0.0"  izz="10.0" />
+			<inertia ixx="${finger_inertia}"  ixy="0"  ixz="0" iyy="${finger_inertia}" iyz="0" izz="${finger_inertia}" />
 			<origin/>
 		</inertial>
@@ -344,10 +336,10 @@
         <parent link="jaco_link_6"/>
         <child link="jaco_finger_link_3"/>
-		<limit lower="-3.1415926535897931" upper="3.1415926535897931" effort="1" velocity="2.0"/>
+		<limit lower="-3.1415926535897931" upper="3.1415926535897931" effort="30" velocity="5"/>
       </joint>
       <link name="jaco_finger_link_3">
 		<inertial>
 			<mass value="0.05"/>
-			<inertia ixx="10.0" ixy="0.0"  ixz="0.0"  iyy="10.0"  iyz="0.0"  izz="10.0" />
+			<inertia ixx="${finger_inertia}"  ixy="0"  ixz="0" iyy="${finger_inertia}" iyz="0" izz="${finger_inertia}" />
 			<origin/>
 		</inertial>

Commit message: standard state made working with gazebo 1.5

File: jaco_driver/jaco_description/urdf/gazebo/jaco.urdf.xacro (robot description, xacro)
@@ -1,14 +1,11 @@
 <?xml version="1.0"?>
-<robot name="jaco"
-  xmlns:xacro="http://ros.org/wiki/xacro">
- <xacro:property name="inertia" value="0.001" />
-  <xacro:property name="finger_inertia" value="0.0001" />
-	<gazebo>
-    <plugin name="gazebo_ros_controller_manager" filename="libgazebo_ros_controller_manager.so">
+<robot name="jaco">
+  <gazebo>
+    <plugin name="gazebo_ros_controller_manager" filename="libgazebo_ros_controller_manager.so" >
       <alwaysOn>true</alwaysOn>
-		<updateRate>1000.0</updateRate>
-		<robotParam>robot_description</robotParam>
+      <updateRate>1000.0</updateRate>
+      <robotParam>robot_description</robotParam>
     </plugin>
-	</gazebo>
+  </gazebo>
 	<include filename="$(find jaco_description)/urdf/gazebo/jaco.gazebo.xacro" />
 	<include filename="$(find jaco_description)/urdf/gazebo/jaco.transmissions.xacro" />
@@ -16,5 +13,4 @@
 	<color rgba="0.2 0.2 0.9 1.0"/>
 	</material>
-	<!--
 	<link name="world"/>
 	<joint name="base_block_joint" type="fixed">
@@ -23,12 +19,11 @@
 		<child link="jaco_base_link" />
 	</joint>
- -->
 	<!-- The base joint & link -->
 	<link name="jaco_base_link">
 		<inertial>
-			<mass value="1" />
+			<mass value="6" />
 			<!--origin xyz="0 0 -0.0525" rpy="0 0 0"/-->
           		<origin xyz="0 0 0.0" rpy="0 0 0"/>
-			<inertia ixx="${inertia}"  ixy="0"  ixz="0" iyy="${inertia}" iyz="0" izz="${inertia}" />
+			<inertia ixx="100"  ixy="0"  ixz="0" iyy="100" iyz="0" izz="100" />
 		</inertial>
 		<visual>
@@ -59,10 +54,10 @@
 		<parent link="jaco_base_link"/>
 		<child link="jaco_link_1"/>
-		<limit lower="-3.1415926535897931" upper="3.1415926535897931" effort="30" velocity="5"/>
+		<limit lower="-3.1415926535897931" upper="3.1415926535897931" effort="1" velocity="2.0"/>
 	</joint>
 	<link name="jaco_link_1">
 		<inertial>
-			<mass value="1" />
-			<inertia ixx="${inertia}"  ixy="0"  ixz="0" iyy="${inertia}" iyz="0" izz="${inertia}" />
+			<mass value="4.5"/>
+			<inertia ixx="100.0" ixy="0.0"  ixz="0.0"  iyy="100.0"  iyz="0.0"  izz="100.0" />
 			<origin/>
 		</inertial>
@@ -93,10 +88,10 @@
 		<parent link="jaco_link_1"/>
 		<child link="jaco_link_2"/>
-		<limit lower="-3.6651914291881" upper="0.57595865315813" effort="30" velocity="5"/>
+		<limit lower="-3.6651914291881" upper="0.57595865315813" effort="1" velocity="3.1415926535897931"/>
 	</joint>
 	<link name="jaco_link_2">
 		<inertial>
-			<mass value="1" />
-			<inertia ixx="${inertia}"  ixy="0"  ixz="0" iyy="${inertia}" iyz="0" izz="${inertia}" />
+			<mass value="3.8"/>
+			<inertia ixx="100.0" ixy="0.0"  ixz="0.0"  iyy="100.0"  iyz="0.0"  izz="100.0" />
 			<origin/>
 		</inertial>
@@ -127,10 +122,10 @@
 		<parent link="jaco_link_2"/>
 		<child link="jaco_link_3"/>
-		<limit lower="-1.221730476396" upper="4.2935099599061" effort="30" velocity="5"/>
+		<limit lower="-1.221730476396" upper="4.2935099599061" effort="1" velocity="3.1415926535897931"/>
 	</joint>
 	<link name="jaco_link_3">
 		<inertial>
-			<mass value="1" />
-			<inertia ixx="${inertia}"  ixy="0"  ixz="0" iyy="${inertia}" iyz="0" izz="${inertia}" />
+			<mass value="2"/>
+			<inertia ixx="100.0" ixy="0.0"  ixz="0.0"  iyy="100.0"  iyz="0.0"  izz="100.0" />
 			<origin/>
 		</inertial>
@@ -161,10 +156,10 @@
 		<parent link="jaco_link_3"/>
 		<child link="jaco_link_4"/>
-		<limit lower="-3.1415926535897931" upper="3.1415926535897931" effort="30" velocity="5"/>
+		<limit lower="-3.1415926535897931" upper="3.1415926535897931" effort="1" velocity="2.0"/>
 	</joint>
 	<link name="jaco_link_4">
 		<inertial>
-			<mass value="1" />
-			<inertia ixx="${inertia}"  ixy="0"  ixz="0" iyy="${inertia}" iyz="0" izz="${inertia}" />
+			<mass value="1.5"/>
+			<inertia ixx="100.0" ixy="0.0"  ixz="0.0"  iyy="100.0"  iyz="0.0"  izz="100.0" />
 			<origin/>
 		</inertial>
@@ -195,10 +190,10 @@
 		<parent link="jaco_link_4"/>
 		<child link="jaco_link_5"/>
-		<limit lower="-3.1415926535897931" upper="3.1415926535897931" effort="30" velocity="5"/>
+		<limit lower="-3.1415926535897931" upper="3.1415926535897931" effort="1" velocity="2.0"/>
 	</joint>
 	<link name="jaco_link_5">
 		<inertial>
 			<mass value="1.0"/>
-			<inertia ixx="${inertia}"  ixy="0"  ixz="0" iyy="${inertia}" iyz="0" izz="${inertia}" />
+			<inertia ixx="100.0" ixy="0.0"  ixz="0.0"  iyy="100.0"  iyz="0.0"  izz="100.0" />
 			<origin/>
 		</inertial>
@@ -231,10 +226,10 @@
 		<parent link="jaco_link_5"/>
 		<child link="jaco_link_6"/>
-		<limit lower="-3.5415926535897931" upper="3.5415926535897931" effort="30" velocity="5"/>
+		<limit lower="-3.5415926535897931" upper="3.5415926535897931" effort="1" velocity="2.0"/>
 	</joint>
 	<link name="jaco_link_6">
 		<inertial>
-			<mass value="0.3"/>
-			<inertia ixx="${inertia}"  ixy="0"  ixz="0" iyy="${inertia}" iyz="0" izz="${inertia}" />
+			<mass value="0.8"/>
+			<inertia ixx="100.0" ixy="0.0"  ixz="0.0"  iyy="100.0"  iyz="0.0"  izz="100.0" />
 			<origin/>
 		</inertial>
@@ -268,10 +263,10 @@
         <parent link="jaco_link_6"/>
         <child link="jaco_finger_link_1"/>
-		<limit lower="-3.1415926535897931" upper="3.1415926535897931" effort="30" velocity="5"/>
+		<limit lower="-3.1415926535897931" upper="3.1415926535897931" effort="1" velocity="2.0"/>
       </joint>
       <link name="jaco_finger_link_1">
 		<inertial>
 			<mass value="0.05"/>
-			<inertia ixx="${finger_inertia}"  ixy="0"  ixz="0" iyy="${finger_inertia}" iyz="0" izz="${finger_inertia}" />
+			<inertia ixx="10.0" ixy="0.0"  ixz="0.0"  iyy="10.0"  iyz="0.0"  izz="10.0" />
 			<origin/>
 		</inertial>
@@ -302,10 +297,10 @@
         <parent link="jaco_link_6"/>
         <child link="jaco_finger_link_2"/>
-		<limit lower="-3.1415926535897931" upper="3.1415926535897931" effort="30" velocity="5"/>
+		<limit lower="-3.1415926535897931" upper="3.1415926535897931" effort="1" velocity="2.0"/>
       </joint>
       <link name="jaco_finger_link_2">
 		<inertial>
 			<mass value="0.05"/>
-			<inertia ixx="${finger_inertia}"  ixy="0"  ixz="0" iyy="${finger_inertia}" iyz="0" izz="${finger_inertia}" />
+			<inertia ixx="10.0" ixy="0.0"  ixz="0.0"  iyy="10.0"  iyz="0.0"  izz="10.0" />
 			<origin/>
 		</inertial>
@@ -336,10 +331,10 @@
         <parent link="jaco_link_6"/>
         <child link="jaco_finger_link_3"/>
-		<limit lower="-3.1415926535897931" upper="3.1415926535897931" effort="30" velocity="5"/>
+		<limit lower="-3.1415926535897931" upper="3.1415926535897931" effort="1" velocity="2.0"/>
       </joint>
       <link name="jaco_finger_link_3">
 		<inertial>
 			<mass value="0.05"/>
-			<inertia ixx="${finger_inertia}"  ixy="0"  ixz="0" iyy="${finger_inertia}" iyz="0" izz="${finger_inertia}" />
+			<inertia ixx="10.0" ixy="0.0"  ixz="0.0"  iyy="10.0"  iyz="0.0"  izz="10.0" />
 			<origin/>
 		</inertial>

Commit message: working but slow

File: jaco_driver/jaco_description/urdf/gazebo/jaco.urdf.xacro (robot description, xacro)
@@ -7,4 +7,5 @@
       <robotParam>robot_description</robotParam>
     </plugin>
+    <turnGravityOff>true</turnGravityOff>
   </gazebo>
 	<include filename="$(find jaco_description)/urdf/gazebo/jaco.gazebo.xacro" />
@@ -13,10 +14,4 @@
 	<color rgba="0.2 0.2 0.9 1.0"/>
 	</material>
-	<link name="world"/>
-	<joint name="base_block_joint" type="fixed">
-		<parent link="world" />
-		<origin xyz="0 0 1" rpy="0 0 0" />
-		<child link="jaco_base_link" />
-	</joint>
 	<!-- The base joint & link -->
 	<link name="jaco_base_link">
