Commit message: changes to make compatible with moveit

File: jaco_driver/jaco_description/urdf/gazebo/jaco.urdf.xacro (robot description, xacro)
@@ -1,12 +1,14 @@
 <?xml version="1.0"?>
-<robot name="jaco">
-  <gazebo>
-    <plugin name="gazebo_ros_controller_manager" filename="libgazebo_ros_controller_manager.so" >
+<robot name="jaco"
+  xmlns:xacro="http://ros.org/wiki/xacro">
+ <xacro:property name="inertia" value="1" />
+  <xacro:property name="finger_inertia" value="1" />
+	<gazebo>
+    <plugin name="gazebo_ros_controller_manager" filename="libgazebo_ros_controller_manager.so">
       <alwaysOn>true</alwaysOn>
-      <updateRate>1000.0</updateRate>
-      <robotParam>robot_description</robotParam>
+		<updateRate>1000.0</updateRate>
+		<robotParam>robot_description</robotParam>
     </plugin>
-    <turnGravityOff>true</turnGravityOff>
-  </gazebo>
+	</gazebo>
 	<include filename="$(find jaco_description)/urdf/gazebo/jaco.gazebo.xacro" />
 	<include filename="$(find jaco_description)/urdf/gazebo/jaco.transmissions.xacro" />
@@ -14,11 +16,19 @@
 	<color rgba="0.2 0.2 0.9 1.0"/>
 	</material>
+	<!--
+	<link name="world"/>
+	<joint name="base_block_joint" type="fixed">
+		<parent link="world" />
+		<origin xyz="0 0 1" rpy="0 0 0" />
+		<child link="jaco_base_link" />
+	</joint>
+ -->
 	<!-- The base joint & link -->
 	<link name="jaco_base_link">
 		<inertial>
-			<mass value="6" />
+			<mass value="1" />
 			<!--origin xyz="0 0 -0.0525" rpy="0 0 0"/-->
           		<origin xyz="0 0 0.0" rpy="0 0 0"/>
-			<inertia ixx="100"  ixy="0"  ixz="0" iyy="100" iyz="0" izz="100" />
+			<inertia ixx="${inertia}"  ixy="0"  ixz="0" iyy="${inertia}" iyz="0" izz="${inertia}" />
 		</inertial>
 		<visual>
@@ -49,10 +59,10 @@
 		<parent link="jaco_base_link"/>
 		<child link="jaco_link_1"/>
-		<limit lower="-3.1415926535897931" upper="3.1415926535897931" effort="1" velocity="2.0"/>
+		<limit lower="-3.1415926535897931" upper="3.1415926535897931" effort="30" velocity="5"/>
 	</joint>
 	<link name="jaco_link_1">
 		<inertial>
-			<mass value="4.5"/>
-			<inertia ixx="100.0" ixy="0.0"  ixz="0.0"  iyy="100.0"  iyz="0.0"  izz="100.0" />
+			<mass value="1" />
+			<inertia ixx="${inertia}"  ixy="0"  ixz="0" iyy="${inertia}" iyz="0" izz="${inertia}" />
 			<origin/>
 		</inertial>
@@ -83,10 +93,10 @@
 		<parent link="jaco_link_1"/>
 		<child link="jaco_link_2"/>
-		<limit lower="-3.6651914291881" upper="0.57595865315813" effort="1" velocity="3.1415926535897931"/>
+		<limit lower="-3.6651914291881" upper="0.57595865315813" effort="30" velocity="5"/>
 	</joint>
 	<link name="jaco_link_2">
 		<inertial>
-			<mass value="3.8"/>
-			<inertia ixx="100.0" ixy="0.0"  ixz="0.0"  iyy="100.0"  iyz="0.0"  izz="100.0" />
+			<mass value="1" />
+			<inertia ixx="${inertia}"  ixy="0"  ixz="0" iyy="${inertia}" iyz="0" izz="${inertia}" />
 			<origin/>
 		</inertial>
@@ -117,10 +127,10 @@
 		<parent link="jaco_link_2"/>
 		<child link="jaco_link_3"/>
-		<limit lower="-1.221730476396" upper="4.2935099599061" effort="1" velocity="3.1415926535897931"/>
+		<limit lower="-1.221730476396" upper="4.2935099599061" effort="30" velocity="5"/>
 	</joint>
 	<link name="jaco_link_3">
 		<inertial>
-			<mass value="2"/>
-			<inertia ixx="100.0" ixy="0.0"  ixz="0.0"  iyy="100.0"  iyz="0.0"  izz="100.0" />
+			<mass value="1" />
+			<inertia ixx="${inertia}"  ixy="0"  ixz="0" iyy="${inertia}" iyz="0" izz="${inertia}" />
 			<origin/>
 		</inertial>
@@ -151,10 +161,10 @@
 		<parent link="jaco_link_3"/>
 		<child link="jaco_link_4"/>
-		<limit lower="-3.1415926535897931" upper="3.1415926535897931" effort="1" velocity="2.0"/>
+		<limit lower="-3.1415926535897931" upper="3.1415926535897931" effort="30" velocity="5"/>
 	</joint>
 	<link name="jaco_link_4">
 		<inertial>
-			<mass value="1.5"/>
-			<inertia ixx="100.0" ixy="0.0"  ixz="0.0"  iyy="100.0"  iyz="0.0"  izz="100.0" />
+			<mass value="1" />
+			<inertia ixx="${inertia}"  ixy="0"  ixz="0" iyy="${inertia}" iyz="0" izz="${inertia}" />
 			<origin/>
 		</inertial>
@@ -185,10 +195,10 @@
 		<parent link="jaco_link_4"/>
 		<child link="jaco_link_5"/>
-		<limit lower="-3.1415926535897931" upper="3.1415926535897931" effort="1" velocity="2.0"/>
+		<limit lower="-3.1415926535897931" upper="3.1415926535897931" effort="30" velocity="5"/>
 	</joint>
 	<link name="jaco_link_5">
 		<inertial>
 			<mass value="1.0"/>
-			<inertia ixx="100.0" ixy="0.0"  ixz="0.0"  iyy="100.0"  iyz="0.0"  izz="100.0" />
+			<inertia ixx="${inertia}"  ixy="0"  ixz="0" iyy="${inertia}" iyz="0" izz="${inertia}" />
 			<origin/>
 		</inertial>
@@ -221,10 +231,10 @@
 		<parent link="jaco_link_5"/>
 		<child link="jaco_link_6"/>
-		<limit lower="-3.5415926535897931" upper="3.5415926535897931" effort="1" velocity="2.0"/>
+		<limit lower="-3.5415926535897931" upper="3.5415926535897931" effort="30" velocity="5"/>
 	</joint>
 	<link name="jaco_link_6">
 		<inertial>
-			<mass value="0.8"/>
-			<inertia ixx="100.0" ixy="0.0"  ixz="0.0"  iyy="100.0"  iyz="0.0"  izz="100.0" />
+			<mass value="0.3"/>
+			<inertia ixx="${inertia}"  ixy="0"  ixz="0" iyy="${inertia}" iyz="0" izz="${inertia}" />
 			<origin/>
 		</inertial>
@@ -251,4 +261,14 @@
 		<turnGravityOff>true</turnGravityOff>
 	</gazebo>
+     <joint name="jaco_gripper_tool_frame_joint" type="fixed">
+      <parent link="jaco_link_6"/>
+      <child link="jaco_gripper_tool_frame" />
+      <origin xyz="0 0 0" rpy="0 ${-M_PI/2} ${M_PI/2}"/>
+    </joint>
+    <link name="jaco_gripper_tool_frame">
+      <!-- This is the coordinate system of the tool (this is the position
+         used in IK etc., relative to the base frame); there is no actual
+         arm part attached to this link -->
+  </link>
 	<!-- first finger joint & link -->
    	<joint name="jaco_finger_joint_1" type="revolute">
@@ -258,13 +278,13 @@
         <parent link="jaco_link_6"/>
         <child link="jaco_finger_link_1"/>
-		<limit lower="-3.1415926535897931" upper="3.1415926535897931" effort="1" velocity="2.0"/>
+		<limit lower="-3.1415926535897931" upper="3.1415926535897931" effort="30" velocity="5"/>
       </joint>
-      <link name="jaco_finger_link_1">
+    <link name="jaco_finger_link_1">
 		<inertial>
 			<mass value="0.05"/>
-			<inertia ixx="10.0" ixy="0.0"  ixz="0.0"  iyy="10.0"  iyz="0.0"  izz="10.0" />
-			<origin/>
-		</inertial>
-        <visual>
+			<inertia ixx="${finger_inertia}"  ixy="0"  ixz="0" iyy="${finger_inertia}" iyz="0" izz="${finger_inertia}" />
+			<origin/>
+		</inertial>
+   <visual>
 			<origin xyz="0 0 0" rpy="0 0 0"/>
           <geometry>
@@ -272,9 +292,9 @@
                 scale="1 1 1"/>
           </geometry>
-        </visual>
+    </visual>
 	<collision>
 			<origin xyz="0 0 0" rpy="0 0 0"/>
 	<geometry>
-            <mesh filename="package://jaco_description/meshes/finger.dae"
+        <mesh filename="package://jaco_description/meshes/finger.dae"
                 scale="1 1 1"/>
 	</geometry>
@@ -292,10 +312,10 @@
         <parent link="jaco_link_6"/>
         <child link="jaco_finger_link_2"/>
-		<limit lower="-3.1415926535897931" upper="3.1415926535897931" effort="1" velocity="2.0"/>
+		<limit lower="-3.1415926535897931" upper="3.1415926535897931" effort="30" velocity="5"/>
       </joint>
       <link name="jaco_finger_link_2">
 		<inertial>
 			<mass value="0.05"/>
-			<inertia ixx="10.0" ixy="0.0"  ixz="0.0"  iyy="10.0"  iyz="0.0"  izz="10.0" />
+			<inertia ixx="${finger_inertia}"  ixy="0"  ixz="0" iyy="${finger_inertia}" iyz="0" izz="${finger_inertia}" />
 			<origin/>
 		</inertial>
@@ -326,10 +346,10 @@
         <parent link="jaco_link_6"/>
         <child link="jaco_finger_link_3"/>
-		<limit lower="-3.1415926535897931" upper="3.1415926535897931" effort="1" velocity="2.0"/>
+		<limit lower="-3.1415926535897931" upper="3.1415926535897931" effort="30" velocity="5"/>
       </joint>
       <link name="jaco_finger_link_3">
 		<inertial>
 			<mass value="0.05"/>
-			<inertia ixx="10.0" ixy="0.0"  ixz="0.0"  iyy="10.0"  iyz="0.0"  izz="10.0" />
+			<inertia ixx="${finger_inertia}"  ixy="0"  ixz="0" iyy="${finger_inertia}" iyz="0" izz="${finger_inertia}" />
 			<origin/>
 		</inertial>

Commit message: switche dto stl files

File: jaco_driver/jaco_description/urdf/gazebo/jaco.urdf.xacro (robot description, xacro)
@@ -36,5 +36,5 @@
 			<!--origin xyz="0 0 -0.0525" rpy="0 0 0"/-->
 			<geometry>
-				<mesh filename="package://jaco_description/meshes/joint_1.dae"
+				<mesh filename="package://jaco_description/meshes/joint_1.stl"
 				scale="0.001 0.001 0.001"/>
 			</geometry>
@@ -43,5 +43,5 @@
 			<!--origin xyz="0 0 -0.0525" rpy="0 0 0"/-->
 			<geometry>
-				<mesh filename="package://jaco_description/meshes/joint_1.dae"
+				<mesh filename="package://jaco_description/meshes/joint_1.stl"
 				scale="0.001 0.001 0.001"/>
 			</geometry>
@@ -71,5 +71,5 @@
 			<origin xyz="0 0 -0.12" rpy="0 0 -1.570796327"/>
 			<geometry>
-				<mesh filename="package://jaco_description/meshes/joint_2.dae"
+				<mesh filename="package://jaco_description/meshes/joint_2.stl"
 				scale="0.001 0.001 0.001"/>
 			</geometry>
@@ -78,5 +78,5 @@
 			<origin xyz="0 0 -0.12" rpy="0 0 -1.570796327"/>
 			<geometry>
-				<mesh filename="package://jaco_description/meshes/joint_2.dae"
+				<mesh filename="package://jaco_description/meshes/joint_2.stl"
 				scale="0.001 0.001 0.001"/>
 			</geometry>
@@ -105,5 +105,5 @@
 			<origin xyz="0 0 0.015" rpy="0 1.570796327 0"/>
 			<geometry>
-				<mesh filename="package://jaco_description/meshes/joint_3.dae"
+				<mesh filename="package://jaco_description/meshes/joint_3.stl"
 				scale="0.001 0.001 0.001"/>
 			</geometry>
@@ -112,5 +112,5 @@
 			<origin xyz="0 0 0.015" rpy="0 1.570796327 0"/>
 			<geometry>
-				<mesh filename="package://jaco_description/meshes/joint_3.dae"
+				<mesh filename="package://jaco_description/meshes/joint_3.stl"
 				scale="0.001 0.001 0.001"/>
 			</geometry>
@@ -139,5 +139,5 @@
 			<origin xyz="0 0 -0.012" rpy="0 1.570796327 1.570796327"/>
 			<geometry>
-				<mesh filename="package://jaco_description/meshes/joint_4.dae"
+				<mesh filename="package://jaco_description/meshes/joint_4.stl"
 				scale="1.000 1.000 1.000"/>
 			</geometry>
@@ -146,5 +146,5 @@
 			<origin xyz="0 0 -0.012" rpy="0 1.570796327 1.570796327"/>
 			<geometry>
-				<mesh filename="package://jaco_description/meshes/joint_4.dae"
+				<mesh filename="package://jaco_description/meshes/joint_4.stl"
 				scale="1.000 1.000 1.000"/>
 			</geometry>
@@ -173,5 +173,5 @@
 			<origin xyz="0 0 -0.042276823" rpy="0 0 -1.570796327"/>
 			<geometry>
-				<mesh filename="package://jaco_description/meshes/joint_5.dae"
+				<mesh filename="package://jaco_description/meshes/joint_5.stl"
 				scale="0.001 0.001 0.001"/>
 			</geometry>
@@ -180,5 +180,5 @@
 			<origin xyz="0 0 -0.042276823" rpy="0 0 -1.570796327"/>
 			<geometry>
-				<mesh filename="package://jaco_description/meshes/joint_5.dae"
+				<mesh filename="package://jaco_description/meshes/joint_5.stl"
 				scale="0.001 0.001 0.001"/>
 			</geometry>
@@ -207,5 +207,5 @@
 			<origin xyz="0 0 -0.042276823" rpy="0 -0.959931089 1.570796327"/>
 			<geometry>
-				<mesh filename="package://jaco_description/meshes/joint_6.dae"
+				<mesh filename="package://jaco_description/meshes/joint_6.stl"
 				scale="0.001 0.001 0.001"/>
 			</geometry>
@@ -214,5 +214,5 @@
 			<origin xyz="0 0 -0.042276823" rpy="0 -0.959931089 1.570796327"/>
 			<geometry>
-				<mesh filename="package://jaco_description/meshes/joint_6.dae"
+				<mesh filename="package://jaco_description/meshes/joint_6.stl"
 				scale="0.001 0.001 0.001"/>
 			</geometry>
@@ -244,5 +244,5 @@
 			<origin xyz="0 0 -0.1850" rpy="0 0 0"/>
 			<geometry>
-				<mesh filename="package://jaco_description/meshes/hand_with_noFinger.dae"
+				<mesh filename="package://jaco_description/meshes/hand_with_noFinger.stl"
 				scale="0.001 0.001 0.001"/>
 			</geometry>
@@ -252,5 +252,5 @@
 			<origin xyz="0 0 -0.1850" rpy="0 0 0"/>
 			<geometry>
-				<mesh filename="package://jaco_description/meshes/hand_with_noFinger.dae"
+				<mesh filename="package://jaco_description/meshes/hand_with_noFinger.stl"
 				scale="0.001 0.001 0.001"/>
 			</geometry>
@@ -264,5 +264,5 @@
       <parent link="jaco_link_6"/>
       <child link="jaco_gripper_tool_frame" />
-      <origin xyz="0 0 0" rpy="0 ${-M_PI/2} ${M_PI/2}"/>
+      <origin xyz="0 0 -0.08" rpy="-0.2 ${-M_PI/2} ${M_PI/2}"/>
     </joint>
     <link name="jaco_gripper_tool_frame">
@@ -289,5 +289,5 @@
 			<origin xyz="0 0 0" rpy="0 0 0"/>
           <geometry>
-            <mesh filename="package://jaco_description/meshes/finger.dae"
+            <mesh filename="package://jaco_description/meshes/finger.stl"
                 scale="1 1 1"/>
           </geometry>
@@ -296,5 +296,5 @@
 			<origin xyz="0 0 0" rpy="0 0 0"/>
 	<geometry>
-        <mesh filename="package://jaco_description/meshes/finger.dae"
+        <mesh filename="package://jaco_description/meshes/finger.stl"
                 scale="1 1 1"/>
 	</geometry>
@@ -323,5 +323,5 @@
 			<origin xyz="0 0 0" rpy="0 0 0"/>
           <geometry>
-            <mesh filename="package://jaco_description/meshes/finger.dae"
+            <mesh filename="package://jaco_description/meshes/finger.stl"
                 scale="1 1 1"/>
           </geometry>
@@ -330,5 +330,5 @@
 			<origin xyz="0 0 0" rpy="0 0 0"/>
 	<geometry>
-            <mesh filename="package://jaco_description/meshes/finger.dae"
+            <mesh filename="package://jaco_description/meshes/finger.stl"
                 scale="1 1 1"/>
 	</geometry>
@@ -357,5 +357,5 @@
 			<origin xyz="0 0 0" rpy="0 0 0"/>
           <geometry>
-            <mesh filename="package://jaco_description/meshes/finger.dae"
+            <mesh filename="package://jaco_description/meshes/finger.stl"
                 scale="1 1 1"/>
           </geometry>
@@ -364,5 +364,5 @@
 			<origin xyz="0 0 0" rpy="0 0 0"/>
 	<geometry>
-            <mesh filename="package://jaco_description/meshes/finger.dae"
+            <mesh filename="package://jaco_description/meshes/finger.stl"
                 scale="1 1 1"/>
 	</geometry>

Commit message: adjust joint limits, adjusted finger positions and gripper frame

File: jaco_driver/jaco_description/urdf/gazebo/jaco.urdf.xacro (robot description, xacro)
@@ -4,4 +4,5 @@
  <xacro:property name="inertia" value="1" />
   <xacro:property name="finger_inertia" value="1" />
+  <xacro:property name="PI" value="3.1415926535897931" />
 	<gazebo>
     <plugin name="gazebo_ros_controller_manager" filename="libgazebo_ros_controller_manager.so">
@@ -59,5 +60,5 @@
 		<parent link="jaco_base_link"/>
 		<child link="jaco_link_1"/>
-		<limit lower="-3.1415926535897931" upper="3.1415926535897931" effort="30" velocity="5"/>
+		<limit lower="${-PI}" upper="${PI}" effort="30" velocity="5"/>
 	</joint>
 	<link name="jaco_link_1">
@@ -93,5 +94,5 @@
 		<parent link="jaco_link_1"/>
 		<child link="jaco_link_2"/>
-		<limit lower="-3.6651914291881" upper="0.57595865315813" effort="30" velocity="5"/>
+		<limit lower="${-PI}" upper="${PI}" effort="30" velocity="5"/>
 	</joint>
 	<link name="jaco_link_2">
@@ -127,5 +128,5 @@
 		<parent link="jaco_link_2"/>
 		<child link="jaco_link_3"/>
-		<limit lower="-1.221730476396" upper="4.2935099599061" effort="30" velocity="5"/>
+		<limit lower="${-PI}" upper="${PI}" effort="30" velocity="5"/>
 	</joint>
 	<link name="jaco_link_3">
@@ -161,5 +162,5 @@
 		<parent link="jaco_link_3"/>
 		<child link="jaco_link_4"/>
-		<limit lower="-3.1415926535897931" upper="3.1415926535897931" effort="30" velocity="5"/>
+		<limit lower="${-PI}" upper="${PI}" effort="30" velocity="5"/>
 	</joint>
 	<link name="jaco_link_4">
@@ -195,5 +196,5 @@
 		<parent link="jaco_link_4"/>
 		<child link="jaco_link_5"/>
-		<limit lower="-3.1415926535897931" upper="3.1415926535897931" effort="30" velocity="5"/>
+		<limit lower="${-PI}" upper="${PI}" effort="30" velocity="5"/>
 	</joint>
 	<link name="jaco_link_5">
@@ -227,9 +228,9 @@
 		<!--origin xyz="0 -0.186174274 0.13036063" rpy="0.959931089 0 0"/-->
 		<origin xyz="0 -0.186174274 0.13036063" rpy="-0.959931089 0 3.1415926535897931"/>
-		<origin xyz="0 0 0" rpy="0 0 -3.14"/>
+		<!--<origin xyz="0 0 0" rpy="0 0 -3.14"/>-->
 		<axis xyz="0 0 -1"/>
 		<parent link="jaco_link_5"/>
 		<child link="jaco_link_6"/>
-		<limit lower="-3.5415926535897931" upper="3.5415926535897931" effort="30" velocity="5"/>
+		<limit lower="${-PI}" upper="${PI}" effort="30" velocity="5"/>
 	</joint>
 	<link name="jaco_link_6">
@@ -241,6 +242,6 @@
 		<visual>
 			<material name="JacoGrey" />
-			<!--origin xyz="0 0 -0.1850" rpy="0 0 -3.1415926535897931"/-->
-			<origin xyz="0 0 -0.1850" rpy="0 0 0"/>
+			<origin xyz="0 0 -0.1850" rpy="0 0 -3.1415926535897931"/>
+			<!--<origin xyz="0 0 -0.1850" rpy="0 0 0"/>      -->
 			<geometry>
 				<mesh filename="package://jaco_description/meshes/hand_with_noFinger.stl"
@@ -249,6 +250,6 @@
 		</visual>
 		<collision>
-			<!--origin xyz="0 0 -0.1850" rpy="0 0 -3.1415926535897931"/-->
-			<origin xyz="0 0 -0.1850" rpy="0 0 0"/>
+			<origin xyz="0 0 -0.1850" rpy="0 0 -3.1415926535897931"/>
+			<!--<origin xyz="0 0 -0.1850" rpy="0 0 0"/>-->
 			<geometry>
 				<mesh filename="package://jaco_description/meshes/hand_with_noFinger.stl"
@@ -264,5 +265,5 @@
       <parent link="jaco_link_6"/>
       <child link="jaco_gripper_tool_frame" />
-      <origin xyz="0 0 -0.08" rpy="-0.2 ${-M_PI/2} ${M_PI/2}"/>
+      <origin xyz="0 0 -0.08" rpy="0.23 ${-3.141592654/2} ${3.141592654/2}"/>
     </joint>
     <link name="jaco_gripper_tool_frame">
@@ -274,9 +275,9 @@
    	<joint name="jaco_finger_joint_1" type="revolute">
         <!--origin xyz="-0.036 -0.021 -0.07" rpy="0 0 0"/--> <!-- changed becuase it look funny in simulation-->
-        <origin xyz="-0.036 -0.021 -0.09" rpy="0 0 0"/>
+        <origin xyz="0.036 -0.021 -0.09" rpy="0 0 ${PI}"/>
         <axis xyz="0 1 0"/>
         <parent link="jaco_link_6"/>
         <child link="jaco_finger_link_1"/>
-		<limit lower="-3.1415926535897931" upper="3.1415926535897931" effort="30" velocity="5"/>
+		<limit lower="0.004" upper="1.044" effort="30" velocity="5"/>
       </joint>
     <link name="jaco_finger_link_1">
@@ -308,9 +309,9 @@
    	<joint name="jaco_finger_joint_2" type="revolute">
         <!--origin xyz="-0.036 0.021 -0.07" rpy="0 0 0"/-->
-	<origin xyz="-0.036 0.021 -0.09" rpy="0 0 0"/>
+	<origin xyz="0.036 0.021 -0.09" rpy="0 0 ${PI + 0.23}"/>
         <axis xyz="0 1 0"/>
         <parent link="jaco_link_6"/>
         <child link="jaco_finger_link_2"/>
-		<limit lower="-3.1415926535897931" upper="3.1415926535897931" effort="30" velocity="5"/>
+		<limit lower="0.004" upper="1.044" effort="30" velocity="5"/>
       </joint>
       <link name="jaco_finger_link_2">
@@ -342,9 +343,9 @@
    	<joint name="jaco_finger_joint_3" type="revolute">
         <!--origin xyz="0.036 -0 -0.07" rpy="0 0 3.14"/-->
-	<origin xyz="0.036 -0 -0.09" rpy="0 0 3.14"/>
+	<origin xyz="-0.036 -0 -0.09" rpy="0 0 0.23"/>
         <axis xyz="0 1 0"/>
         <parent link="jaco_link_6"/>
         <child link="jaco_finger_link_3"/>
-		<limit lower="-3.1415926535897931" upper="3.1415926535897931" effort="30" velocity="5"/>
+		<limit lower="0.004" upper="1.044" effort="30" velocity="5"/>
       </joint>
       <link name="jaco_finger_link_3">
