Commit message: start.lauch to use jaco.urdf

File: jaco_driver/jaco_description/urdf/gazebo/jaco.urdf (robot description, URDF)
Before this commit: robot jaco, 11 links, 10 joints
Links:
- added link base_link
Joints:
- added joint base_joint: type fixed, parent base_link, child jaco_base_link, origin xyz=0 0 0
- joint jaco_finger_joint_1: limit lower=-3.1415926535897931 upper=3.1415926535897931 effort=30 velocity=5 -> lower=0.004 upper=1.044 effort=30 velocity=5; origin xyz=-0.036 -0.021 -0.09 rpy=0 0 0 -> xyz=0.036 -0.021 -0.09 rpy=0 0 3.14159265359
- joint jaco_finger_joint_2: limit lower=-3.1415926535897931 upper=3.1415926535897931 effort=30 velocity=5 -> lower=0.004 upper=1.044 effort=30 velocity=5; origin xyz=-0.036 0.021 -0.09 rpy=0 0 0 -> xyz=0.036 0.021 -0.09 rpy=0 0 3.37159265359
- joint jaco_finger_joint_3: limit lower=-3.1415926535897931 upper=3.1415926535897931 effort=30 velocity=5 -> lower=0.004 upper=1.044 effort=30 velocity=5; origin xyz=0.036 -0 -0.09 rpy=0 0 3.14 -> xyz=-0.036 -0 -0.09 rpy=0 0 0.23
- joint jaco_gripper_tool_frame_joint: origin xyz=0 0 -0.08 rpy=-0.2 -1.570796327 1.570796327 -> xyz=0 0 -0.08 rpy=0.23 -1.570796327 1.570796327
- joint jaco_joint_1: limit lower=-3.1415926535897931 upper=3.1415926535897931 effort=30 velocity=5 -> lower=-3.14159265359 upper=3.14159265359 effort=30 velocity=5
- joint jaco_joint_2: limit lower=-3.6651914291881 upper=0.57595865315813 effort=30 velocity=5 -> lower=-3.14159265359 upper=3.14159265359 effort=30 velocity=5
- joint jaco_joint_3: limit lower=-1.221730476396 upper=4.2935099599061 effort=30 velocity=5 -> lower=-3.14159265359 upper=3.14159265359 effort=30 velocity=5
- joint jaco_joint_4: limit lower=-3.1415926535897931 upper=3.1415926535897931 effort=30 velocity=5 -> lower=-3.14159265359 upper=3.14159265359 effort=30 velocity=5
- joint jaco_joint_5: limit lower=-3.1415926535897931 upper=3.1415926535897931 effort=30 velocity=5 -> lower=-3.14159265359 upper=3.14159265359 effort=30 velocity=5
- joint jaco_joint_6: limit lower=-3.5415926535897931 upper=3.5415926535897931 effort=30 velocity=5 -> lower=-3.14159265359 upper=3.14159265359 effort=30 velocity=5
